Commit message: Motion problem solved and navigation works

File: cyber_robt/urdf/cyber_robt_base.urdf.xacro (robot description, xacro)
@@ -77,7 +77,7 @@
         rpy="0 0 0" />
       <geometry>
-        <!-- <cylinder radius="0.06" length="0.05"/> -->
-        <mesh
-          filename="package://cyber_robt/meshes/W_B_L.STL" />
+        <cylinder radius="0.06" length="0.06"/>
+        <!-- <mesh
+          filename="package://cyber_robt/meshes/W_B_L.STL" /> -->
       </geometry>
     </collision>
@@ -95,10 +95,10 @@
     <axis
       xyz="0 0 1" />
-    <!-- <limit
+    <limit
       effort="10"
       velocity="10" />
     <dynamics
       damping="0.1"
-      friction="0.1" /> -->
+      friction="0.1" />
     <mimic joint="W_F_L_joint"/>
   </joint>
@@ -138,7 +138,7 @@
         rpy="0 0 0" />
       <geometry>
-        <!-- <cylinder radius="0.06" length="0.05"/> -->
-        <mesh
-          filename="package://cyber_robt/meshes/W_F_L.STL" />
+        <cylinder radius="0.06" length="0.06"/>
+        <!-- <mesh
+          filename="package://cyber_robt/meshes/W_F_L.STL" /> -->
       </geometry>
     </collision>
@@ -156,10 +156,10 @@
     <axis
       xyz="0 0 1" />
-    <!-- <limit
+    <limit
       effort="10"
       velocity="10" />
     <dynamics
       damping="0.1"
-      friction="0.1" /> -->
+      friction="0.1" />
   </joint>
   <link
@@ -198,7 +198,7 @@
         rpy="0 0 0" />
       <geometry>
-        <!-- <cylinder radius="0.06" length="0.05"/> -->
-        <mesh
-          filename="package://cyber_robt/meshes/W_B_R.STL" />
+        <cylinder radius="0.06" length="0.06"/>
+        <!-- <mesh
+          filename="package://cyber_robt/meshes/W_B_R.STL" /> -->
       </geometry>
     </collision>
@@ -209,5 +209,5 @@
     <origin
       xyz="-0.19374 -0.16473 0.01975"
-      rpy="-1.5708 0 0" />
+      rpy="1.5708 0 0" />
     <parent
       link="base_link" />
@@ -215,11 +215,11 @@
       link="W_B_R" />
     <axis
-      xyz="0 0 1" />
-    <!-- <limit
+      xyz="0 0 -1" />
+    <limit
       effort="10"
       velocity="10" />
     <dynamics
       damping="0.1"
-      friction="0.1" /> -->
+      friction="0.1" />
     <mimic joint="W_F_R_joint"/>
   </joint>
@@ -259,7 +259,7 @@
         rpy="0 0 0" />
       <geometry>
-        <!-- <cylinder radius="0.06" length="0.05"/> -->
-        <mesh
-          filename="package://cyber_robt/meshes/W_F_R.STL" />
+        <cylinder radius="0.06" length="0.06"/>
+        <!-- <mesh
+          filename="package://cyber_robt/meshes/W_F_R.STL" /> -->
       </geometry>
     </collision>
@@ -270,5 +270,5 @@
     <origin
       xyz="0.17626 -0.16473 0.01975"
-      rpy="-1.5708 0 0" />
+      rpy="1.5708 0 0" />
     <parent
       link="base_link" />
@@ -276,11 +276,11 @@
       link="W_F_R" />
     <axis
-      xyz="0 0 1" />
-    <!-- <limit
+      xyz="0 0 -1" />
+    <limit
       effort="10"
       velocity="10" />
     <dynamics
       damping="0.1"
-      friction="0.1" /> -->
+      friction="0.1" />
   </joint>
   <link

File: cyber_robt/urdf/ignition_plugins.xacro (robot description, xacro)
@@ -80,5 +80,5 @@
     <plugin filename="libgz-sim-diff-drive-system" name="gz::sim::systems::DiffDrive">
         <!-- Update rate in Hz -->
-        <update_rate>50</update_rate>
+        <update_rate>20</update_rate>
         <!-- wheels -->
         <left_joint>W_F_L_joint</left_joint>
@@ -87,8 +87,9 @@
         <right_joint>W_B_R_joint</right_joint>
         <!-- kinematics -->
-        <wheel_separation>0.35</wheel_separation>
+        <wheel_separation>0.4</wheel_separation>
         <wheel_radius>0.06</wheel_radius> <!-- replace with actual value -->
         <!-- limits -->
         <max_acceleration>5.0</max_acceleration>
+        <max_velocity>10.0</max_velocity>
         <!-- input -->
         <topic>/cmd_vel</topic>

Commit message: Motion mismatch solved and navigation needs some tuning

File: cyber_robt/urdf/cyber_robt_base.urdf.xacro (robot description, xacro)
@@ -49,5 +49,5 @@
         rpy="0 0 0" />
       <mass
-        value="0.3" />
+        value="0.110835075707755" />
       <inertia
         ixx="0.000173950330336761"
@@ -77,5 +77,5 @@
         rpy="0 0 0" />
       <geometry>
-        <cylinder radius="0.06" length="0.06"/>
+        <cylinder radius="0.06" length="0.05"/>
         <!-- <mesh
           filename="package://cyber_robt/meshes/W_B_L.STL" /> -->
@@ -110,5 +110,5 @@
         rpy="0 0 0" />
       <mass
-        value="0.3" />
+        value="0.110835075707755" />
       <inertia
         ixx="0.000173950330312339"
@@ -138,5 +138,5 @@
         rpy="0 0 0" />
       <geometry>
-        <cylinder radius="0.06" length="0.06"/>
+        <cylinder radius="0.06" length="0.05"/>
         <!-- <mesh
           filename="package://cyber_robt/meshes/W_F_L.STL" /> -->
@@ -170,5 +170,5 @@
         rpy="0 0 0" />
       <mass
-        value="0.3" />
+        value="0.110835075707755" />
       <inertia
         ixx="0.000173950330329626"
@@ -198,5 +198,5 @@
         rpy="0 0 0" />
       <geometry>
-        <cylinder radius="0.06" length="0.06"/>
+        <cylinder radius="0.06" length="0.05"/>
         <!-- <mesh
           filename="package://cyber_robt/meshes/W_B_R.STL" /> -->
@@ -231,5 +231,5 @@
         rpy="0 0 0" />
       <mass
-        value="0.3" />
+        value="0.110835075707755" />
       <inertia
         ixx="0.000173950330336794"
@@ -259,5 +259,5 @@
         rpy="0 0 0" />
       <geometry>
-        <cylinder radius="0.06" length="0.06"/>
+        <cylinder radius="0.06" length="0.05"/>
         <!-- <mesh
           filename="package://cyber_robt/meshes/W_F_R.STL" /> -->

File: cyber_robt/urdf/ignition_plugins.xacro (robot description, xacro)
@@ -5,8 +5,8 @@
         filename="ignition-gazebo-joint-state-publisher-system"/>
 -->
-      <!--   <plugin
+        <plugin
             filename="gz-sim-physics-system"
             name="gz::sim::systems::Physics">
-        </plugin>-->
+        </plugin>
      <plugin
         filename="gz-sim-scene-broadcaster-system"
@@ -80,5 +80,5 @@
     <plugin filename="libgz-sim-diff-drive-system" name="gz::sim::systems::DiffDrive">
         <!-- Update rate in Hz -->
-        <update_rate>20</update_rate>
+        <update_rate>100</update_rate>
         <!-- wheels -->
         <left_joint>W_F_L_joint</left_joint>
@@ -87,5 +87,5 @@
         <right_joint>W_B_R_joint</right_joint>
         <!-- kinematics -->
-        <wheel_separation>0.4</wheel_separation>
+        <wheel_separation>0.9</wheel_separation>
         <wheel_radius>0.06</wheel_radius> <!-- replace with actual value -->
         <!-- limits -->
